Commit message: replace wx200 by wx250s as boris arm

File: mani_skill/assets/robots/boris/boris.urdf (robot description, URDF)
Before this commit: robot shark-v1, 54 links, 53 joints
Links:
- removed link boris_arm/ee_arm_link
- removed link boris_arm/ee_gripper_link
- removed link boris_arm/fingers_link
- removed link boris_arm/fingers_yaw_link
- removed link boris_arm/forearm_link
- removed link boris_arm/gripper_bar_link
- removed link boris_arm/gripper_link
- removed link boris_arm/gripper_prop_link
- removed link boris_arm/left_finger_link
- removed link boris_arm/right_finger_link
- removed link boris_arm/shoulder_link
- removed link boris_arm/upper_arm_link
- removed link boris_arm/wrist_link
- added link ee_arm_link, mass 0.001
- added link ee_gripper_link, mass 0.001
- added link fingers_link, mass 0.001
- added link gripper_bar_link, mass 0.034199; collision mesh filename=meshes_wx250s/WXSA-250-M-9-Gripper-Bar.stl scale=0.001 0.001 0.001; visual mesh filename=meshes_wx250s/WXSA-250-M-9-Gripper-Bar.obj scale=0.001 0.001 0.001
- added link gripper_link, mass 0.072885; collision mesh filename=meshes_wx250s/WXSA-250-M-7-Gripper.stl scale=0.001 0.001 0.001; visual mesh filename=meshes_wx250s/WXSA-250-M-7-Gripper.obj scale=0.001 0.001 0.001
- added link gripper_prop_link, mass 0.00434; visual mesh filename=meshes_wx250s/WXSA-250-M-8-Gripper-Prop.obj scale=0.001 0.001 0.001
- added link left_finger_link, mass 0.016246; collision mesh filename=meshes_wx250s/WXSA-250-M-10-Finger.stl scale=0.001 0.001 0.001; visual mesh filename=meshes_wx250s/WXSA-250-M-10-Finger.obj scale=0.001 0.001 0.001
- added link lower_forearm_link, mass 0.220991; collision mesh filename=meshes_wx250s/WXSA-250-M-5-LF.stl scale=0.001 0.001 0.001; visual mesh filename=meshes_wx250s/WXSA-250-M-5-LF.obj scale=0.001 0.001 0.001
- added link right_finger_link, mass 0.016246; collision mesh filename=meshes_wx250s/WXSA-250-M-10-Finger.stl scale=0.001 0.001 0.001; visual mesh filename=meshes_wx250s/WXSA-250-M-10-Finger.obj scale=0.001 0.001 0.001
- added link shoulder_link, mass 0.480879; collision mesh filename=meshes_wx250s/WXSA-250-M-2-Shoulder.stl scale=0.001 0.001 0.001; visual mesh filename=meshes_wx250s/WXSA-250-M-2-Shoulder.obj scale=0.001 0.001 0.001
- added link upper_arm_link, mass 0.430811; collision mesh filename=meshes_wx250s/WXSA-250-M-3-UA.stl scale=0.001 0.001 0.001; visual mesh filename=meshes_wx250s/WXSA-250-M-3-UA.obj scale=0.001 0.001 0.001
- added link upper_forearm_link, mass 0.234589; collision mesh filename=meshes_wx250s/WXSA-250-M-4-UF.stl scale=0.001 0.001 0.001; visual mesh filename=meshes_wx250s/WXSA-250-M-4-UF.obj scale=0.001 0.001 0.001
- added link wrist_link, mass 0.084957; collision mesh filename=meshes_wx250s/WXSA-250-M-6-Wrist.stl scale=0.001 0.001 0.001; visual mesh filename=meshes_wx250s/WXSA-250-M-6-Wrist.obj scale=0.001 0.001 0.001
- link boris_arm/base_link: mass 0.379673 -> 0.538736; geometry collision mesh filename=meshes_wx250s/WXSA-250-M-1-Base.stl scale=0.001 0.001 0.001; visual mesh filename=meshes_wx250s/WXSA-250-M-1-Base.obj scale=0.001 0.001 0.001
Joints:
- removed joint wrist_yaw
- added joint forearm_roll: type revolute, parent upper_forearm_link, child lower_forearm_link, origin xyz=0.175 0 0 rpy=0 0 0, axis 1 0 0, limit lower=-3.141582653589793 upper=3.141582653589793 effort=2 velocity=3.141592653589793
- joint ee_arm: child boris_arm/ee_arm_link -> ee_arm_link; parent boris_arm/gripper_link -> gripper_link
- joint ee_bar: child boris_arm/fingers_link -> fingers_link; parent boris_arm/gripper_bar_link -> gripper_bar_link
- joint ee_gripper: child boris_arm/ee_gripper_link -> ee_gripper_link; limit lower=-3.14 upper=3.14 effort=1 velocity=3.141592653589793 -> (none); parent boris_arm/fingers_yaw_link -> fingers_link
- joint elbow: child boris_arm/forearm_link -> upper_forearm_link; limit lower=-2.251 upper=2.251 effort=76.94 velocity=1.571 -> lower=-2.1467549799530254 upper=1.6057029118347832 effort=15 velocity=3.141592653589793; origin xyz=0.05 0 0.2 rpy=0 0 0 -> xyz=0.04975 0 0.25 rpy=0 0 0; parent boris_arm/upper_arm_link -> upper_arm_link
- joint gripper: child boris_arm/gripper_prop_link -> gripper_prop_link; limit effort=1 velocity=3.141592653589793 -> (none); parent boris_arm/ee_arm_link -> ee_arm_link; type continuous -> fixed
- joint gripper_bar: child boris_arm/gripper_bar_link -> gripper_bar_link; parent boris_arm/ee_arm_link -> ee_arm_link
- joint head_pan_joint: type revolute -> fixed
- joint head_tilt_joint: type revolute -> fixed
- joint horizontal_neck_joint: type revolute -> fixed
- joint jaw_joint: type revolute -> fixed
- joint left_eye_horizontal_joint: type revolute -> fixed
- joint left_eye_vertical_joint: type revolute -> fixed
- joint left_finger: axis 0 -1 0 -> 0 1 0; child boris_arm/left_finger_link -> left_finger_link; limit lower=0.0 upper=0.037 effort=60 velocity=0.05 -> lower=0.015 upper=0.037 effort=5 velocity=1; origin xyz=0.03 0.037 0 rpy=0 0 0 -> xyz=0 0 0 rpy=0 0 0; parent boris_arm/fingers_link -> fingers_link
- joint left_inferior_eyelid_joint: type revolute -> fixed
- joint left_rotacional_eyebrow_joint: type revolute -> fixed
- joint left_superior_eyelid_joint: type revolute -> fixed
- joint left_vertical_eyebrow_joint: type prismatic -> fixed
- joint left_wheel_joint: type continuous -> fixed
- joint right_eye_horizontal_joint: type revolute -> fixed
- joint right_eye_vertical_joint: type revolute -> fixed
- joint right_finger: axis 0 1 0 -> 0 -1 0; child boris_arm/right_finger_link -> right_finger_link; limit lower=0.00 upper=0.037 effort=60 velocity=0.05 -> lower=0.015 upper=0.037 effort=5 velocity=1; mimic joint=left_finger -> (none); origin xyz=0.03 -0.037 0 rpy=0 0 0 -> xyz=0 0 0 rpy=0 0 0; parent boris_arm/fingers_link -> fingers_link
- joint right_inferior_eyelid_joint: type revolute -> fixed
- joint right_rotacional_eyebrow_joint: type revolute -> fixed
- joint right_superior_eyelid_joint: type revolute -> fixed
- joint right_vertical_eyebrow_joint: type prismatic -> fixed
- joint right_wheel_joint: type continuous -> fixed
- joint shoulder: child boris_arm/upper_arm_link -> upper_arm_link; limit lower=-1.221 upper=1.518 effort=131.76 velocity=1.454 -> lower=-1.8849555921538759 upper=1.9896753472735358 effort=20 velocity=3.141592653589793; parent boris_arm/shoulder_link -> shoulder_link
- joint vertical_neck_joint: type revolute -> fixed
- joint waist: child boris_arm/shoulder_link -> shoulder_link; limit lower=-1.6056 upper=1.6056 effort=33.82 velocity=1.256 -> lower=-3.141592653589793 upper=3.141592653589793 effort=10 velocity=3.141592653589793; origin xyz=0 0 0.066175 rpy=0 0 0 -> xyz=0 0 0.072 rpy=0 0 0
- joint wrist_angle: child boris_arm/wrist_link -> wrist_link; limit lower=-2.251 upper=2.251 effort=66.18 velocity=1.521 -> lower=-1.7453292519943295 upper=2.1467549799530254 effort=5 velocity=3.141592653589793; origin xyz=0.2 0 0 rpy=0 1.57 0 -> xyz=0.075 0 0 rpy=0 0 0; parent boris_arm/forearm_link -> lower_forearm_link
- joint wrist_rotate: child boris_arm/gripper_link -> gripper_link; limit lower=-2.251 upper=2.251 effort=29.35 velocity=1.571 -> lower=-3.141582653589793 upper=3.141582653589793 effort=1 velocity=3.141592653589793; parent boris_arm/wrist_link -> wrist_link
